Commit message: 10.01

File: src/a1_description/urdf/a1.urdf (robot description, URDF)
Before this commit: robot a1, 23 links, 22 joints
Links:
- added link world
Joints:
- added joint base_static_joint: type fixed, parent world, child base, origin xyz=0 0 0 rpy=0 0 0
- joint FL_calf_joint: limit lower=-2.69653369433 upper=-0.916297857297 effort=33.5 velocity=21 -> lower=-3 upper=4 effort=33.5 velocity=21
- joint FL_hip_joint: limit lower=-0.802851455917 upper=0.802851455917 effort=33.5 velocity=21 -> lower=-3 upper=3 effort=33.5 velocity=21
- joint FL_thigh_joint: limit lower=-1.0471975512 upper=4.18879020479 effort=33.5 velocity=21 -> lower=-3 upper=4.18879020479 effort=33.5 velocity=21
- joint FR_calf_joint: limit lower=-2.69653369433 upper=-0.916297857297 effort=33.5 velocity=21 -> lower=-3.69653369433 upper=3 effort=33.5 velocity=21
- joint FR_thigh_joint: limit lower=-1.0471975512 upper=4.18879020479 effort=33.5 velocity=21 -> lower=-3 upper=4.18879020479 effort=33.5 velocity=21
- joint RL_calf_joint: limit lower=-2.69653369433 upper=-0.916297857297 effort=33.5 velocity=21 -> lower=-3 upper=4 effort=33.5 velocity=21
- joint RL_hip_joint: limit lower=-0.802851455917 upper=0.802851455917 effort=33.5 velocity=21 -> lower=-3 upper=3 effort=33.5 velocity=21
- joint RL_thigh_joint: limit lower=-1.0471975512 upper=4.18879020479 effort=33.5 velocity=21 -> lower=-3 upper=4.18879020479 effort=33.5 velocity=21
- joint RR_calf_joint: limit lower=-2.69653369433 upper=-0.916297857297 effort=33.5 velocity=21 -> lower=-3 upper=4 effort=33.5 velocity=21
- joint RR_hip_joint: limit lower=-0.802851455917 upper=0.802851455917 effort=33.5 velocity=21 -> lower=-3 upper=3 effort=33.5 velocity=21
- joint RR_thigh_joint: limit lower=-1.0471975512 upper=4.18879020479 effort=33.5 velocity=21 -> lower=-3 upper=4.18879020479 effort=33.5 velocity=21
